Commit message: Updated URDF

File: description/urdf/kartyb_description.urdf.xacro (robot description, xacro)
@@ -20,10 +20,10 @@
   </link>
   <!-- BASE_FOOTPRINT LINK -->
-  <joint name="base_footprint_joint" type="fixed">
-      <parent link="base_link"/>
-      <child link="base_footprint"/>
+  <joint name="${prefix}base_footprint_joint" type="fixed">
+      <parent link="${prefix}base_link"/>
+      <child link="${prefix}base_footprint"/>
       <origin xyz="0 0 0" rpy="0 0 0"/>
   </joint>
-  <link name="base_footprint">
+  <link name="${prefix}base_footprint">
   </link>
   <!-- Chassis Link -->
@@ -51,8 +51,8 @@
     </xacro:inertial_box>
   </link>
-  <gazebo reference="chassis">
+  <gazebo reference="${prefix}chassis">
       <material>Gazebo/Green</material>
   </gazebo>
-  <!-- Steering Left Pivot Link -->
+  Steering Left Pivot Link
   <joint name="${prefix}steering_left_pivot_joint" type="continuous">
     <parent link="${prefix}base_link"/>

File: description/urdf/lidar.xacro (robot description, xacro)
@@ -1,4 +1,5 @@
 <?xml version="1.0"?>
 <robot xmlns:xacro="http://www.ros.org/wiki/xacro" >
+<xacro:macro name="diffbot" params="prefix">
     <joint name="laser_joint" type="fixed">
         <parent link="base_link"/>
@@ -50,3 +51,4 @@
         </sensor>
     </gazebo>
+</xacro:macro>
 </robot>
