Commit message: Updated URDF

File: description/urdf/kartyb_description_diffdrive.urdf.xacro (robot description, xacro)
@@ -54,30 +54,4 @@
       <material>Gazebo/Green</material>
   </gazebo>
-  Steering Left Pivot Link
-  <joint name="steering_left_pivot_joint" type="continuous">
-    <parent link="base_link"/>
-    <child link="steering_left_pivot"/>
-    <origin xyz="${wheel_pos_front} ${wheel_pivot_pos_front} 0.02" rpy="0 0 0"/>
-    <axis xyz="0 0 1"/>
-  </joint>
-  <link name="steering_left_pivot">
-    <visual>
-        <geometry>
-            <cylinder length="0.1" radius="0.025"/>
-        </geometry>
-        <material name="white"/>
-    </visual>
-    <collision>
-        <geometry>
-            <cylinder length="0.1" radius="0.025"/>
-        </geometry>
-    </collision>
-    <xacro:inertial_cylinder mass="${wheel_mass}" length="0.1" radius="0.025">
-          <origin xyz="0 0 0" rpy="0 0 0"/>
-    </xacro:inertial_cylinder>
-  </link>
-  <gazebo reference="steering_left_pivot">
-      <material>Gazebo/White</material>
-  </gazebo>
   <!-- left wheel front Link -->
   <joint name="left_wheel_joint" type="continuous">
@@ -105,30 +79,4 @@
   <gazebo reference="left_wheel">
       <material>Gazebo/Black</material>
-  </gazebo>
-  <!-- Steering Right Pivot Link -->
-  <joint name="steering_right_pivot_joint" type="continuous">
-    <parent link="base_link"/>
-    <child link="steering_right_pivot"/>
-    <origin xyz="${wheel_pos_front} ${-wheel_pivot_pos_front} 0.02" rpy="0 0 ${PI}"/>
-    <axis xyz="0 0 1"/>
-  </joint>
-  <link name="steering_right_pivot">
-    <visual>
-        <geometry>
-            <cylinder length="0.1" radius="0.025"/>
-        </geometry>
-        <material name="white"/>
-    </visual>
-    <collision>
-        <geometry>
-            <cylinder length="0.1" radius="0.025"/>
-        </geometry>
-    </collision>
-    <xacro:inertial_cylinder mass="${wheel_mass}" length="0.1" radius="0.025">
-          <origin xyz="0 0 0" rpy="0 0 0"/>
-    </xacro:inertial_cylinder>
-  </link>
-  <gazebo reference="steering_right_pivot">
-      <material>Gazebo/White</material>
   </gazebo>
   <!-- right wheel front Link -->
@@ -158,56 +106,4 @@
       <material>Gazebo/Black</material>
   </gazebo>
-  <!-- left wheel rear Link -->
-  <joint name="left_wheel_rear_joint" type="continuous">
-    <parent link="base_link"/>
-    <child link="left_wheel_rear"/>
-    <origin xyz="-${wheel_pos_rear} ${chassis_width/2 + wheel_len/2} 0" rpy="-${PI/2} 0 0"/>
-    <axis xyz="0 0 1"/>
-  </joint>
-  <link name="left_wheel_rear">
-    <visual>
-      <geometry>
-        <cylinder length="${wheel_len}" radius="${wheel_radius}"/>
-      </geometry>
-      <material name="black"/>
-    </visual>
-    <collision>
-      <geometry>
-        <cylinder length="${wheel_len}" radius="${wheel_radius}"/>
-      </geometry>
-    </collision>
-    <xacro:inertial_cylinder mass="${wheel_mass}" length="${wheel_len}" radius="${wheel_radius}">
-          <origin xyz="0 0 0" rpy="0 0 0"/>
-    </xacro:inertial_cylinder>
-  </link>
-  <gazebo reference="left_wheel_rear">
-      <material>Gazebo/Black</material>
-  </gazebo>
-  <!-- right wheel rear Link -->
-  <joint name="right_wheel_rear_joint" type="continuous">
-    <parent link="base_link"/>
-    <child link="right_wheel_rear"/>
-    <origin xyz="-${wheel_pos_rear} -${chassis_width/2 + wheel_len/2} 0" rpy="${PI/2} 0 0"/>
-    <axis xyz="0 0 -1"/>
-  </joint>
-  <link name="right_wheel_rear">
-    <visual>
-      <geometry>
-        <cylinder length="${wheel_len}" radius="${wheel_radius}"/>
-      </geometry>
-      <material name="black"/>
-    </visual>
-    <collision>
-      <geometry>
-        <cylinder length="${wheel_len}" radius="${wheel_radius}"/>
-      </geometry>
-    </collision>
-    <xacro:inertial_cylinder mass="${wheel_mass}" length="${wheel_len}" radius="${wheel_radius}">
-          <origin xyz="0 0 0" rpy="0 0 0"/>
-    </xacro:inertial_cylinder>
-  </link>
-  <gazebo reference="right_wheel_rear">
-      <material>Gazebo/Black</material>
-  </gazebo>
   </xacro:macro>
 </robot>

Commit message: Updated urdf origins and orientations

File: description/urdf/kartyb_description_diffdrive.urdf.xacro (robot description, xacro)
@@ -58,6 +58,6 @@
     <parent link="base_link"/>
     <child link="left_wheel"/>
-    <origin xyz="${chassis_length/2} ${chassis_width/2} 0" rpy="-${PI/2} 0 0"/>
-    <axis xyz="0 0 1"/>
+    <origin xyz="${chassis_length/2} ${chassis_width/2} 0" rpy="${PI/2} 0 0"/>
+    <axis xyz="0 0 -1"/>
   </joint>
   <link name="left_wheel">
@@ -84,6 +84,6 @@
     <parent link="base_link"/>
     <child link="right_wheel"/>
-    <origin xyz="${chassis_length/2} ${-chassis_width/2} 0" rpy="${PI/2} 0 0"/>
-    <axis xyz="0 0 -1"/>
+    <origin xyz="${chassis_length/2} ${-chassis_width/2} 0" rpy="-${PI/2} 0 0"/>
+    <axis xyz="0 0 1"/>
   </joint>
   <link name="right_wheel">

File: description/urdf/lidar.xacro (robot description, xacro)
@@ -1,8 +1,9 @@
 <?xml version="1.0"?>
 <robot xmlns:xacro="http://www.ros.org/wiki/xacro" >
+    <xacro:property name="PI" value="3.1415926535897931"/>
     <joint name="laser_joint" type="fixed">
         <parent link="base_link"/>
         <child link="laser_frame"/>
-        <origin xyz="-0.12 0 0.4" rpy="0 0 3.1415926535897931"/>
+        <origin xyz="-0.12 0 0.4" rpy="0 0 -${PI/2}"/>
     </joint>
     <link name="laser_frame">

Commit message: Updated urdf description - left wheel orientation

File: description/urdf/kartyb_description_diffdrive.urdf.xacro (robot description, xacro)
@@ -58,6 +58,6 @@
     <parent link="chassis"/>
     <child link="left_wheel"/>
-    <origin xyz="${chassis_length} ${chassis_width/2} -0.07" rpy="${PI/2} 0 0"/>
-    <axis xyz="0 0 -1"/>
+    <origin xyz="${chassis_length} ${chassis_width/2} -0.07" rpy="-${PI/2} 0 0"/>
+    <axis xyz="0 0 1"/>
   </joint>
   <link name="left_wheel">

Commit message: updated description left wheel

File: description/urdf/kartyb_description_diffdrive.urdf.xacro (robot description, xacro)
@@ -58,5 +58,5 @@
     <parent link="chassis"/>
     <child link="left_wheel"/>
-    <origin xyz="${chassis_length} ${chassis_width/2} -0.07" rpy="-${PI/2} 0 0"/>
+    <origin xyz="${chassis_length} ${chassis_width/2} -0.07" rpy="${PI/2} 0 0"/>
     <axis xyz="0 0 1"/>
   </joint>

Commit message: Updated decription urdf

File: description/urdf/kartyb_description_diffdrive.urdf.xacro (robot description, xacro)
@@ -31,5 +31,5 @@
     <parent link="base_link"/>
     <child link="chassis"/>
-    <origin xyz="-${chassis_length/2} 0 ${chassis_base_offset}"/>
+    <origin xyz="${-chassis_length/2} 0 ${chassis_base_offset}"/>
   </joint>
   <link name="chassis">
@@ -58,5 +58,5 @@
     <parent link="chassis"/>
     <child link="left_wheel"/>
-    <origin xyz="${chassis_length} ${chassis_width/2} -0.07" rpy="${PI/2} 0 0"/>
+    <origin xyz="${chassis_length} ${chassis_width/2} -0.07" rpy="-${PI/2} 0 0"/>
     <axis xyz="0 0 1"/>
   </joint>
@@ -84,6 +84,6 @@
     <parent link="chassis"/>
     <child link="right_wheel"/>
-    <origin xyz="${chassis_length} ${-chassis_width/2} -0.07" rpy="-${PI/2} 0 0"/>
-    <axis xyz="0 0 1"/>
+    <origin xyz="${chassis_length} ${-chassis_width/2} -0.07" rpy="${PI/2} 0 0"/>
+    <axis xyz="0 0 -1"/>
   </joint>
   <link name="right_wheel">

Commit message: updated controller params

File: description/urdf/kartyb_description_diffdrive.urdf.xacro (robot description, xacro)
@@ -59,5 +59,5 @@
     <child link="left_wheel"/>
     <origin xyz="${chassis_length} ${chassis_width/2} -0.07" rpy="-${PI/2} 0 0"/>
-    <axis xyz="0 0 1"/>
+    <axis xyz="0 0 -1"/>
   </joint>
   <link name="left_wheel">

Commit message: updated urdf

File: description/urdf/kartyb_description_diffdrive.urdf.xacro (robot description, xacro)
@@ -56,5 +56,5 @@
   <!-- left wheel front Link -->
   <joint name="left_wheel_joint" type="continuous">
-    <parent link="chassis"/>
+    <parent link="base_link"/>
     <child link="left_wheel"/>
     <origin xyz="${chassis_length} ${chassis_width/2} -0.07" rpy="-${PI/2} 0 0"/>
@@ -82,5 +82,5 @@
   <!-- right wheel front Link -->
   <joint name="right_wheel_joint" type="continuous">
-    <parent link="chassis"/>
+    <parent link="base_link"/>
     <child link="right_wheel"/>
     <origin xyz="${chassis_length} ${-chassis_width/2} -0.07" rpy="${PI/2} 0 0"/>

Commit message: Added slam toolbox params

File: description/urdf/kartyb_description_diffdrive.urdf.xacro (robot description, xacro)
@@ -56,8 +56,8 @@
   <!-- left wheel front Link -->
   <joint name="left_wheel_joint" type="continuous">
-    <parent link="base_link"/>
+    <parent link="chassis"/>
     <child link="left_wheel"/>
     <origin xyz="${chassis_length} ${chassis_width/2} -0.07" rpy="-${PI/2} 0 0"/>
-    <axis xyz="0 0 -1"/>
+    <axis xyz="0 0 1"/>
   </joint>
   <link name="left_wheel">
@@ -82,5 +82,5 @@
   <!-- right wheel front Link -->
   <joint name="right_wheel_joint" type="continuous">
-    <parent link="base_link"/>
+    <parent link="chassis"/>
     <child link="right_wheel"/>
     <origin xyz="${chassis_length} ${-chassis_width/2} -0.07" rpy="${PI/2} 0 0"/>
