Commit message: updated urdf

File: description/ros2_control/gazebo.ros2_control.xacro (robot description, xacro)
@@ -2,9 +2,9 @@
 <robot xmlns:xacro="http://www.ros.org/wiki/xacro">
     <xacro:macro name="diffbot_ros2_control" params="name prefix">
-        <ros2_control name="GazeboSystem" type="system">
+        <ros2_control name="${name}" type="system">
             <hardware>
                 <plugin>gazebo_ros2_control/GazeboSystem</plugin>
             </hardware>
-            <joint name="left_wheel_joint">
+            <joint name="${prefix}left_wheel_joint">
                 <command_interface name="velocity">
                     <param name="min">-10</param>
@@ -14,5 +14,5 @@
                 <state_interface name="position"/>
             </joint>
-            <joint name="right_wheel_joint">
+            <joint name="${prefix}right_wheel_joint">
                 <command_interface name="velocity">
                     <param name="min">-10</param>

File: description/urdf/diffbot.urdf.xacro (robot description, xacro)
@@ -10,8 +10,7 @@
   <xacro:include filename="$(find ros2_control_demo_example_2)/urdf/materials.xacro" />
   <!-- Import diffbot ros2_control description -->
-  <!-- <xacro:include filename="$(find ros2_control_demo_example_2)/ros2_control/diffbot.ros2_control.xacro" /> -->
-  <xacro:include filename="$(find ros2_control_demo_example_2)/ros2_control/gazebo.ros2_control.xacro" />
+  <xacro:include filename="$(find ros2_control_demo_example_2)/ros2_control/diffbot.ros2_control.xacro" />
+  <!-- <xacro:include filename="$(find ros2_control_demo_example_2)/ros2_control/gazebo.ros2_control.xacro" /> -->
   <xacro:diffbot prefix="$(arg prefix)" />
-  <xacro:diffbot_ros2_control
-    name="DiffBot" prefix="$(arg prefix)" use_mock_hardware="$(arg use_mock_hardware)"/>
+  <xacro:diffbot_ros2_control name="DiffBot" prefix="$(arg prefix)" use_mock_hardware="$(arg use_mock_hardware)"/>
 </robot>

File: description/urdf/lidar.xacro (robot description, xacro)
@@ -2,10 +2,10 @@
 <robot xmlns:xacro="http://www.ros.org/wiki/xacro" >
 <xacro:macro name="diffbot" params="prefix">
-    <joint name="laser_joint" type="fixed">
-        <parent link="base_link"/>
-        <child link="laser_frame"/>
+    <joint name="${prefix}laser_joint" type="fixed">
+        <parent link="${prefix}base_link"/>
+        <child link="${prefix}laser_frame"/>
         <origin xyz="0.1 0 0.125" rpy="0 0 3.1415926535897931"/>
     </joint>
-    <link name="laser_frame">
+    <link name="${prefix}laser_frame">
         <visual>
             <geometry>

Commit message: Have gazebo working now for kartyB diffbot

File: description/ros2_control/gazebo.ros2_control.xacro (robot description, xacro)
@@ -1,10 +1,9 @@
 <?xml version="1.0"?>
 <robot xmlns:xacro="http://www.ros.org/wiki/xacro">
-    <xacro:macro name="diffbot_ros2_control" params="name prefix">
-        <ros2_control name="${name}" type="system">
+        <ros2_control name="RoboGazebo" type="system">
             <hardware>
                 <plugin>gazebo_ros2_control/GazeboSystem</plugin>
             </hardware>
-            <joint name="${prefix}left_wheel_joint">
+            <joint name="left_wheel_joint">
                 <command_interface name="velocity">
                     <param name="min">-10</param>
@@ -14,5 +13,5 @@
                 <state_interface name="position"/>
             </joint>
-            <joint name="${prefix}right_wheel_joint">
+            <joint name="right_wheel_joint">
                 <command_interface name="velocity">
                     <param name="min">-10</param>
@@ -29,4 +28,3 @@
             </plugin>
         </gazebo>
-    </xacro:macro>
 </robot>

File: description/urdf/diffbot.urdf.xacro (robot description, xacro)
@@ -5,6 +5,6 @@
   <xacro:include filename="$(find ros2_control_demo_example_2)/urdf/inertial_macros.xacro" />
   <xacro:include filename="$(find ros2_control_demo_example_2)/urdf/kartyb_description_diffdrive.urdf.xacro" />
-  <!-- <xacro:include filename="$(find ros2_control_demo_example_2)/urdf/test_robot_description.urdf.xacro" /> -->
-  <!-- <xacro:include filename="$(find ros2_control_demo_example_2)/urdf/lidar.xacro" /> -->
+  <xacro:include filename="$(find ros2_control_demo_example_2)/urdf/kartyb_face.urdf.xacro" />
+  <xacro:include filename="$(find ros2_control_demo_example_2)/urdf/lidar.xacro" />
   <!-- Import Rviz colors -->
   <xacro:include filename="$(find ros2_control_demo_example_2)/urdf/materials.xacro" />
@@ -13,4 +13,4 @@
   <!-- <xacro:include filename="$(find ros2_control_demo_example_2)/ros2_control/gazebo.ros2_control.xacro" /> -->
   <xacro:diffbot prefix="$(arg prefix)" />
-  <xacro:diffbot_ros2_control name="DiffBot" prefix="$(arg prefix)" use_mock_hardware="$(arg use_mock_hardware)"/>
+  <!-- <xacro:diffbot_ros2_control name="DiffBot" prefix="$(arg prefix)" use_mock_hardware="$(arg use_mock_hardware)"/> -->
 </robot>

File: description/urdf/kartyb_description_diffdrive.urdf.xacro (robot description, xacro)
@@ -39,5 +39,5 @@
             <box size="${chassis_length} ${chassis_width} ${chassis_height}"/>
         </geometry>
-        <material name="white"/>
+        <material name="green"/>
     </visual>
     <collision>
@@ -58,5 +58,5 @@
     <parent link="base_link"/>
     <child link="left_wheel"/>
-    <origin xyz="0 0.045 -0.02" rpy="-${PI/2} 0 0"/>
+    <origin xyz="${chassis_length/2} ${chassis_width/2} 0" rpy="-${PI/2} 0 0"/>
     <axis xyz="0 0 1"/>
   </joint>
@@ -84,5 +84,5 @@
     <parent link="base_link"/>
     <child link="right_wheel"/>
-    <origin xyz="0 0.045 -0.02" rpy="-${PI/2} 0 0"/>
+    <origin xyz="${chassis_length/2} ${-chassis_width/2} 0" rpy="${PI/2} 0 0"/>
     <axis xyz="0 0 -1"/>
   </joint>
@@ -106,4 +106,32 @@
       <material>Gazebo/Black</material>
   </gazebo>
+  <!-- rear caster Link -->
+  <joint name="caster_wheel_joint" type="fixed">
+    <parent link="base_link"/>
+    <child link="caster_wheel"/>
+    <origin xyz="${(-chassis_length/2)+(wheel_radius)} 0 0" rpy="-${PI/2} 0 0"/>
+    <axis xyz="0 0 -1"/>
+  </joint>
+  <link name="caster_wheel">
+    <visual>
+      <geometry>
+        <cylinder length="${wheel_len}" radius="${wheel_radius}"/>
+      </geometry>
+      <material name="black"/>
+    </visual>
+    <collision>
+      <geometry>
+        <cylinder length="${wheel_len}" radius="${wheel_radius}"/>
+      </geometry>
+    </collision>
+    <xacro:inertial_cylinder mass="${wheel_mass}" length="${wheel_len}" radius="${wheel_radius}">
+          <origin xyz="0 0 0" rpy="0 0 0"/>
+    </xacro:inertial_cylinder>
+  </link>
+  <gazebo reference="caster_wheel">
+      <material>Gazebo/Black</material>
+      <mu1 value="0.001"/>
+      <mu2 value="0.001"/>
+  </gazebo>
   </xacro:macro>
 </robot>

File: description/urdf/lidar.xacro (robot description, xacro)
@@ -1,11 +1,10 @@
 <?xml version="1.0"?>
 <robot xmlns:xacro="http://www.ros.org/wiki/xacro" >
-<xacro:macro name="diffbot" params="prefix">
-    <joint name="${prefix}laser_joint" type="fixed">
-        <parent link="${prefix}base_link"/>
-        <child link="${prefix}laser_frame"/>
-        <origin xyz="0.1 0 0.125" rpy="0 0 3.1415926535897931"/>
+    <joint name="laser_joint" type="fixed">
+        <parent link="base_link"/>
+        <child link="laser_frame"/>
+        <origin xyz="-0.12 0 0.4" rpy="0 0 3.1415926535897931"/>
     </joint>
-    <link name="${prefix}laser_frame">
+    <link name="laser_frame">
         <visual>
             <geometry>
@@ -51,4 +50,3 @@
         </sensor>
     </gazebo>
-</xacro:macro>
 </robot>
