Commit message: Updated ros2 control xacro

File: description/ros2_control/diffbot.ros2_control.xacro (robot description, xacro)
@@ -50,14 +50,12 @@
         <state_interface name="velocity"/>
       </joint>
-      <joint name="${prefix}steering_left_pivot_joint">
+      <!-- <joint name="${prefix}steering_left_pivot_joint">
         <command_interface name="position"/>
         <state_interface name="position"/>
-        <!-- <state_interface name="velocity"/> -->
       </joint>
       <joint name="${prefix}steering_right_pivot_joint">
         <command_interface name="position"/>
         <state_interface name="position"/>
-        <!-- <state_interface name="velocity"/> -->
-      </joint>
+      </joint> -->
     </ros2_control>
   </xacro:macro>

Commit message: Updates for rviz config

File: description/ros2_control/diffbot.ros2_control.xacro (robot description, xacro)
@@ -50,5 +50,5 @@
         <state_interface name="velocity"/>
       </joint>
-      <!-- <joint name="${prefix}steering_left_pivot_joint">
+      <joint name="${prefix}steering_left_pivot_joint">
         <command_interface name="position"/>
         <state_interface name="position"/>
@@ -57,5 +57,5 @@
         <command_interface name="position"/>
         <state_interface name="position"/>
-      </joint> -->
+      </joint>
     </ros2_control>
   </xacro:macro>

File: description/urdf/diffbot.urdf.xacro (robot description, xacro)
@@ -11,4 +11,5 @@
   <!-- Import diffbot ros2_control description -->
   <xacro:include filename="$(find ros2_control_demo_example_2)/ros2_control/diffbot.ros2_control.xacro" />
+  <xacro:include filename="$(find ros2_control_demo_example_2)/ros2_control/gazebo.ros2_control.xacro" />
   <xacro:diffbot prefix="$(arg prefix)" />
   <xacro:diffbot_ros2_control

Commit message: updated urdf

File: description/ros2_control/diffbot.ros2_control.xacro (robot description, xacro)
@@ -50,5 +50,5 @@
         <state_interface name="velocity"/>
       </joint>
-      <joint name="${prefix}steering_left_pivot_joint">
+      <!-- <joint name="${prefix}steering_left_pivot_joint">
         <command_interface name="position"/>
         <state_interface name="position"/>
@@ -57,5 +57,5 @@
         <command_interface name="position"/>
         <state_interface name="position"/>
-      </joint>
+      </joint> -->
     </ros2_control>
   </xacro:macro>

Commit message: Urdf updates

File: description/ros2_control/diffbot.ros2_control.xacro (robot description, xacro)
@@ -40,10 +40,10 @@
         </hardware>
       </xacro:if>
-      <joint name="${prefix}left_wheel_joint">
+      <joint name="left_wheel_joint">
         <command_interface name="velocity"/>
         <state_interface name="position"/>
         <state_interface name="velocity"/>
       </joint>
-      <joint name="${prefix}right_wheel_joint">
+      <joint name="right_wheel_joint">
         <command_interface name="velocity"/>
         <state_interface name="position"/>

Commit message: removed macro tags

File: description/ros2_control/diffbot.ros2_control.xacro (robot description, xacro)
@@ -1,7 +1,5 @@
 <?xml version="1.0"?>
 <robot xmlns:xacro="http://www.ros.org/wiki/xacro">
-  <xacro:macro name="diffbot_ros2_control" params="name prefix use_mock_hardware">
-    <ros2_control name="${name}" type="system">
-      <xacro:unless value="${use_mock_hardware}">
+    <ros2_control name="diffbot_ros2_control" type="system">
         <hardware>
           <plugin>ros2_control_demo_example_2/DiffBotSystemHardware</plugin>
@@ -33,11 +31,4 @@
           <param name="ddsm115_right_wheel_id">4</param>
         </hardware>
-      </xacro:unless>
-      <xacro:if value="${use_mock_hardware}">
-        <hardware>
-          <plugin>mock_components/GenericSystem</plugin>
-          <param name="calculate_dynamics">true</param>
-        </hardware>
-      </xacro:if>
       <joint name="left_wheel_joint">
         <command_interface name="velocity"/>
@@ -59,4 +50,3 @@
       </joint> -->
     </ros2_control>
-  </xacro:macro>
 </robot>

Commit message: Updated Gazebo and the URDF files

File: description/ros2_control/diffbot.ros2_control.xacro (robot description, xacro)
@@ -5,5 +5,5 @@
           <plugin>ros2_control_demo_example_2/DiffBotSystemHardware</plugin>
           <!-- ... -->
-          <!-- MCU Settings -->
+          <!-- MCU Settings - Used for serial comms to Servos -->
           <param name="steering_left_name">steering_left_pivot_joint</param>
           <param name="steering_right_name">steering_right_pivot_joint</param>
@@ -41,4 +41,5 @@
         <state_interface name="velocity"/>
       </joint>
+      <!-- Uncomment below when using Ackermann Controller -->
       <!-- <joint name="${prefix}steering_left_pivot_joint">
         <command_interface name="position"/>

File: description/urdf/diffbot.urdf.xacro (robot description, xacro)
@@ -7,9 +7,10 @@
   <xacro:include filename="$(find ros2_control_demo_example_2)/urdf/kartyb_face.urdf.xacro" />
   <xacro:include filename="$(find ros2_control_demo_example_2)/urdf/lidar.xacro" />
+  <xacro:include filename="$(find ros2_control_demo_example_2)/urdf/camera.xacro" />
   <!-- Import Rviz colors -->
   <xacro:include filename="$(find ros2_control_demo_example_2)/urdf/materials.xacro" />
   <!-- Import diffbot ros2_control description -->
-  <xacro:include filename="$(find ros2_control_demo_example_2)/ros2_control/diffbot.ros2_control.xacro" />
-  <!-- <xacro:include filename="$(find ros2_control_demo_example_2)/ros2_control/gazebo.ros2_control.xacro" /> -->
+  <!-- <xacro:include filename="$(find ros2_control_demo_example_2)/ros2_control/diffbot.ros2_control.xacro" /> -->
+  <xacro:include filename="$(find ros2_control_demo_example_2)/ros2_control/gazebo.ros2_control.xacro" />
   <xacro:diffbot prefix="$(arg prefix)" />
   <!-- <xacro:diffbot_ros2_control name="DiffBot" prefix="$(arg prefix)" use_mock_hardware="$(arg use_mock_hardware)"/> -->

File: description/urdf/kartyb_description_diffdrive.urdf.xacro (robot description, xacro)
@@ -5,8 +5,8 @@
   <xacro:property name="PI" value="3.1415926535897931"/>
   <xacro:property name="chassis_mass" value="0.8" /> <!-- arbitrary value for base mass -->
-  <xacro:property name="chassis_width" value="0.3" />
-  <xacro:property name="chassis_length" value="0.35" />
-  <xacro:property name="chassis_height" value="0.32" />
-  <xacro:property name="chassis_base_offset" value="0.07" />
+  <xacro:property name="chassis_width" value="0.22" />
+  <xacro:property name="chassis_length" value="0.28" />
+  <xacro:property name="chassis_height" value="0.22" />
+  <xacro:property name="chassis_base_offset" value="0.12" />
   <xacro:property name="wheel_mass" value="0.3" /> <!-- arbitrary value for wheel mass -->
   <xacro:property name="wheel_len" value="0.040" />
@@ -56,7 +56,7 @@
   <!-- left wheel front Link -->
   <joint name="left_wheel_joint" type="continuous">
-    <parent link="base_link"/>
+    <parent link="chassis"/>
     <child link="left_wheel"/>
-    <origin xyz="${chassis_length/2} ${chassis_width/2} 0" rpy="${PI/2} 0 0"/>
+    <origin xyz="${chassis_length} ${chassis_width/2} -0.07" rpy="${PI/2} 0 0"/>
     <axis xyz="0 0 -1"/>
   </joint>
@@ -82,7 +82,7 @@
   <!-- right wheel front Link -->
   <joint name="right_wheel_joint" type="continuous">
-    <parent link="base_link"/>
+    <parent link="chassis"/>
     <child link="right_wheel"/>
-    <origin xyz="${chassis_length/2} ${-chassis_width/2} 0" rpy="-${PI/2} 0 0"/>
+    <origin xyz="${chassis_length} ${-chassis_width/2} -0.07" rpy="-${PI/2} 0 0"/>
     <axis xyz="0 0 1"/>
   </joint>
@@ -108,7 +108,7 @@
   <!-- rear caster Link -->
   <joint name="caster_wheel_joint" type="fixed">
-    <parent link="base_link"/>
+    <parent link="chassis"/>
     <child link="caster_wheel"/>
-    <origin xyz="${(-chassis_length/2)+(wheel_radius)} 0 0" rpy="-${PI/2} 0 0"/>
+    <origin xyz="${wheel_radius} 0 -0.07" rpy="-${PI/2} 0 0"/>
     <axis xyz="0 0 -1"/>
   </joint>

File: description/urdf/kartyb_face.urdf.xacro (robot description, xacro)
@@ -2,12 +2,12 @@
 <robot xmlns:xacro="http://www.ros.org/wiki/xacro">
   <xacro:property name="PI" value="3.1415926535897931"/>
-  <xacro:property name="chassis_width" value="0.3" />
-  <xacro:property name="chassis_length" value="0.35" />
-  <xacro:property name="chassis_height" value="0.32" />
+  <xacro:property name="chassis_width" value="0.22" />
+  <xacro:property name="chassis_length" value="0.28" />
+  <xacro:property name="chassis_height" value="0.22" />
   <!-- kartyB Face Link -->
   <joint name="face_joint" type="fixed">
     <parent link="chassis"/>
     <child link="face"/>
-    <origin xyz="${chassis_length} 0 0.2" rpy="0 -${PI/2} 0"/>
+    <origin xyz="${chassis_length} 0 0.15" rpy="0 -${PI/2} 0"/>
     <axis xyz="0 0 -1"/>
   </joint>

File: description/urdf/lidar.xacro (robot description, xacro)
@@ -2,8 +2,11 @@
 <robot xmlns:xacro="http://www.ros.org/wiki/xacro" >
     <xacro:property name="PI" value="3.1415926535897931"/>
+    <xacro:property name="chassis_width" value="0.22" />
+    <xacro:property name="chassis_length" value="0.28" />
+    <xacro:property name="chassis_height" value="0.22" />
     <joint name="laser_joint" type="fixed">
-        <parent link="base_link"/>
+        <parent link="chassis"/>
         <child link="laser_frame"/>
-        <origin xyz="-0.12 0 0.4" rpy="0 0 -${PI/2}"/>
+        <origin xyz="0.025 0 ${chassis_height + 0.03}" rpy="0 0 -${PI/2}"/>
     </joint>
     <link name="laser_frame">
@@ -16,8 +19,8 @@
         <collision>
             <geometry>
-                <cylinder radius="0.05" length="0.04"/>
+                <cylinder radius="0.03" length="0.04"/>
             </geometry>
         </collision>
-        <xacro:inertial_cylinder mass="0.1" length="0.04" radius="0.05">
+        <xacro:inertial_cylinder mass="0.1" length="0.04" radius="0.03">
             <origin xyz="0 0 0" rpy="0 0 0"/>
         </xacro:inertial_cylinder>
